Commit message: -

File: src/description/robot.urdf (robot description, URDF)
Before this commit: robot two_wheel, 5 links, 4 joints
Joints:
- joint drivewhl_l_joint: limit lower=-0.999999 upper=0.999999 effort=5 velocity=1 -> lower=-999999 upper=999999 effort=5 velocity=1
- joint drivewhl_r_joint: limit lower=-0.999999 upper=0.999999 effort=5 velocity=1 -> lower=-999999 upper=999999 effort=5 velocity=1
